File: v0.1/PCBs/raveniung-board.kicad_pcb (KiCad board)
At the start: 2 copper layers, 287 x 111.7 mm, 92 parts

Commit message: add routed v0.1 PCBs
Parts:
- moved D35 87.8 mm to (238.7, 172.5), turned to 26 degrees
- moved S35 84.6 mm to (236.5, 168.0), turned to 26 degrees
- moved D34 70.0 mm to (159.7, 161.6), turned to -15 degrees
- moved S34 67.0 mm to (161.0, 156.8), turned to -15 degrees
- moved MH1 9.22 mm to (208.0, 168.0)
- moved S33 8.68 mm to (179.5, 168.0), turned to -26 degrees
- moved D36 8.64 mm to (256.2, 161.6), turned to 15 degrees
- moved D16 8.50 mm to (176.7, 102.9)
- moved D23 8.50 mm to (294.5, 88.3)
- moved MH9 8.50 mm to (325.2, 98.1)
- moved D24 8.50 mm to (281.6, 124.4)
- moved S18 8.50 mm to (335.2, 100.2)
- moved D18 8.50 mm to (336.1, 105.2)
- moved S17 8.50 mm to (338.5, 119.0)
- moved D13 8.50 mm to (158.8, 94.9)
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Connections:
- D33 pad 2: default_default -> inner_thumb
- D34 pad 2: mirror_default_default -> reachy_thumb
- D35 pad 2: default_default -> mirror_inner_thumb
- D36 pad 2: mirror_default_default -> mirror_reachy_thumb
- S33 pad 1: default_default -> inner_thumb
- S34 pad 1: mirror_default_default -> reachy_thumb
- S34 pad 2: COL2 -> COL0
- S35 pad 1: default_default -> mirror_inner_thumb
- S35 pad 2: COL0 -> COL2
- S36 pad 1: mirror_default_default -> mirror_reachy_thumb
Routing:
- net COL0: track 378.5 -> 293.9 mm, vias 0 -> 1
- net COL5: track 281.5 -> 253.6 mm, vias 0 -> 1
- net mirror_default_default: track 21.7 -> 0.00 mm
- net default_default: track 21.4 -> 0.00 mm
- net ROW6: track 165.8 -> 184.7 mm
- net COL3: track 345.3 -> 327.6 mm
- net COL2: track 354.6 -> 338.0 mm
- net COL4: track 300.2 -> 286.4 mm, vias 2 -> 1
- net mirror_reachy_thumb: track 0.00 -> 11.1 mm
- net mirror_inner_thumb: track 0.00 -> 11.0 mm
- net inner_thumb: track 0.00 -> 10.7 mm
- net reachy_thumb: track 0.00 -> 10.7 mm
- net COL1: track 324.3 -> 315.4 mm
- net ROW1: track 146.8 -> 155.6 mm
- net ROW4: track 153.5 -> 159.0 mm
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Other:
- board size 287 x 111.7 mm -> 287 x 114.2 mm
