File: v0.2/PCBs/raveniung-board.kicad_pcb (KiCad board)
At the start: 2 copper layers, 304 x 114.2 mm, 92 parts

Commit message: Add finished kicad pcb inclusive gerbers
Parts:
- moved S10 6.86 mm to (151.3, 82.5)
- moved S15 6.86 mm to (183.8, 117.2)
- moved S24 6.86 mm to (307.2, 120.0)
- moved D17 6.86 mm to (365.9, 124.4)
- moved S32 6.86 mm to (264.9, 98.5)
- moved D7 6.86 mm to (130.9, 88.8)
- moved D2 6.86 mm to (89.4, 105.7)
- moved D19 6.86 mm to (347.2, 127.7)
- moved S14 6.86 mm to (180.5, 136.0)
- moved MCU1 6.86 mm to (226.0, 106.1)
- moved S11 6.86 mm to (162.6, 128.0)
- moved S31 6.86 mm to (268.2, 117.2)
- moved D26 6.86 mm to (301.5, 87.4)
- moved D32 6.86 mm to (265.7, 103.4)
- moved S13 6.86 mm to (169.2, 90.5)
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Routing:
- net COL2: track 0.00 -> 365.5 mm, vias 0 -> 2
- net COL3: track 0.00 -> 347.6 mm, vias 0 -> 2
- net COL0: track 0.00 -> 331.9 mm, vias 0 -> 1
- net COL1: track 0.00 -> 325.3 mm, vias 0 -> 1
- net COL4: track 0.00 -> 307.7 mm, vias 0 -> 1
- net COL5: track 0.00 -> 274.0 mm, vias 0 -> 1
- net ROW6: track 0.00 -> 206.5 mm
- net ROW2: track 0.00 -> 181.2 mm
- net ROW5: track 0.00 -> 173.2 mm
- net ROW4: track 0.00 -> 165.4 mm
- net ROW1: track 0.00 -> 163.9 mm
- net ROW3: track 0.00 -> 130.1 mm
- net ROW0: track 0.00 -> 102.9 mm
- net GND: track 0.00 -> 90.7 mm, vias 0 -> 1
- net RDY: track 0.00 -> 41.9 mm, vias 0 -> 1
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