File: v0.2/PCBs/raveniung-top-plate.kicad_pcb (KiCad board)
At the start: 2 copper layers, 304 x 114.2 mm, 11 parts

Commit message: Add finished kicad top plate inclusive gerbers
Other:
- outline, holes or cut-outs redrawn
- board text added: "raveniung v0.2"
- board text removed: "raveniung ver0.1"
